File: PCB-Eagle/VFD-Power.brd (EAGLE design)
At the start: 83.5 x 27.9 mm, 24 parts, among them IC1 74HC132D, IC3 ZXBM5210

Commit message: fixed Up Converter R9/R10 twist, adjusted values for 50V
Parts:
- R2: value 39 -> 1.5k
- R3: value 1k -> 39
