File: PCB-KiCad/GP1294-Teens4.kicad_pcb (KiCad board)
At the start: 2 copper layers, 225 x 48 mm, 31 parts, among them IC1 74132D, IC2 XL6009, IC3 ZXBM5210, SW1 RotaryEncoder_Switch, SW2 RotaryEncoder_Switch, SW3 SW_Push, SW4 SW_Push, U3 R-78B5.0-2.0

Commit message: Progress on GP1294 board..
Parts:
- removed SW2: RotaryEncoder_Switch, Rotary_Encoder:RotaryEncoder_Alps_EC12E_Vertical_H20mm
- added SW5: RotaryEncoder_Switch, Rotary_Encoder:RotaryEncoder_Alps_EC12E-Switch_Vertical_H20mm, B.Cu at (34.0, 56.8)
- added SW6: RotaryEncoder_Switch, Rotary_Encoder:RotaryEncoder_Alps_EC12E-Switch_Vertical_H20mm, B.Cu at (237.9, 57.0)
- SW1: value RotaryEncoder_Switch -> SW_Push; footprint Rotary_Encoder:RotaryEncoder_Alps_EC12E_Vertical_H20mm -> Button_Switch_THT:SW_PUSH-12mm_Wuerth-430476085716
- SW3, SW4: moved to B.Cu
- moved SW4 166.8 mm to (57.5, 47.0), turned to 180 degrees
- moved SW3 37.3 mm to (57.5, 32.5), turned to 180 degrees
- moved SW1 6.69 mm to (45.0, 61.5), turned to 0 degrees
- moved U2 2.97 mm to (124.0, 27.0)
- moved POWER0 1.00 mm to (217.8, 28.0)
Connections:
- U2 pad 7: unconnected-(U2-5-Pad7) -> Net-(U2-5)
Routing:
- net Net-(U1-CLK): track 0.00 -> 67.3 mm
- net Net-(U1-CS): track 50.5 -> 51.2 mm
Other:
- board size 225 x 48 mm -> 225 x 48.5 mm

Commit message: GP1294 progress..
Parts:
- removed SW6: RotaryEncoder_Switch, Rotary_Encoder:RotaryEncoder_Alps_EC12E-Switch_Vertical_H20mm
- added Case1: ~, VFDs-Library:CaseDD, F.Cu at (150.0, 100.0)
- added ENC1: RotaryEncoder_Switch, Rotary_Encoder:RotaryEncoder_Alps_EC12E-Switch_Vertical_H20mm, B.Cu at (221.0, 122.5)
- added ENC2: RotaryEncoder_Switch, Rotary_Encoder:RotaryEncoder_Alps_EC12E-Switch_Vertical_H20mm, B.Cu at (94.0, 122.5)
- added SW2: SW_Push, Button_Switch_THT:SW_PUSH-12mm_Wuerth-430476085716, B.Cu at (137.5, 104.5)
- SW1: moved to B.Cu
- SW5: value RotaryEncoder_Switch -> SW_Push; footprint Rotary_Encoder:RotaryEncoder_Alps_EC12E-Switch_Vertical_H20mm -> Button_Switch_THT:SW_PUSH-12mm_Wuerth-430476085716
- moved SW5 166.5 mm to (193.5, 104.5), turned to 180 degrees
- moved POWER0 155.3 mm to (66.8, 64.2), turned to -90 degrees
- moved L3 140.1 mm to (71.8, 91.2)
- moved IC2 140.0 mm to (71.7, 106.3)
- moved C3 137.8 mm to (80.5, 65.1)
- moved C2 130.9 mm to (91.5, 83.5)
- moved SW4 130.8 mm to (175.0, 104.5)
- moved C6 130.8 mm to (80.5, 77.9), turned to 180 degrees
- moved SW3 122.2 mm to (156.2, 104.5)
- moved U2 121.6 mm to (238.5, 67.8), turned to -90 degrees
- moved U1 102.0 mm to (150.0, 75.0)
- moved L2 88.4 mm to (98.0, 67.5)
- moved U3 88.4 mm to (85.5, 90.4), turned to 0 degrees
- moved SW1 85.6 mm to (119.0, 104.5), turned to 180 degrees
- moved C7 63.5 mm to (135.0, 74.9)
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Other:
- board size 225 x 48.5 mm -> 178.5 x 99.4 mm
- board text added: "inputs"
- board text added: "links"
- board text added: "outputs"
- board text added: "rechts"
- board text added: "x=150"
- board text added: "y=100"

Commit message: GP1294 progress...
Parts:
- removed POWER0: MA06-1, VFD-Power:MA06-1
- added R6: 100, Resistor_SMD:R_0603_1608Metric, F.Cu at (199.1, 80.1)
- added R7: 100, Resistor_SMD:R_0603_1608Metric, F.Cu at (199.1, 82.6)
- added R8: 100, Resistor_SMD:R_0603_1608Metric, F.Cu at (199.1, 85.1)
- added R9: 100, Resistor_SMD:R_0603_1608Metric, F.Cu at (199.1, 87.6)
- added U4: ~, FreeDSP:FreeDSP-allinone, B.Cu at (220.8, 150.1)
- moved SW1 17.9 mm to (119.0, 122.4)
- moved SW2 17.9 mm to (137.5, 122.4)
- moved SW3 17.9 mm to (156.2, 122.4)
- moved SW4 17.9 mm to (175.0, 122.4)
- moved SW5 17.9 mm to (193.5, 122.4)
Connections:
- FILLAMENT0 pad 1: /Power/F1 -> F1
- FILLAMENT0 pad 2: /Power/F1 -> F1
- FILLAMENT0 pad 3: /Power/F2 -> F2
- FILLAMENT0 pad 4: /Power/F2 -> F2
- IC3 pad 1: /Power/F1 -> F1
- R5 pad 1: /Power/F2 -> F2
- U1 pad 1: unconnected-(U1-F+-Pad1) -> F1
- U1 pad 28: unconnected-(U1-F--Pad28) -> F2
- U2 pad 20: unconnected-(U2-A4-Pad20) -> /LRCLK1
- U2 pad 21: unconnected-(U2-A5-Pad21) -> /BCLK1
- U2 pad 8: unconnected-(U2-6-Pad8) -> /OUT1
- U2 pad 9: unconnected-(U2-7-Pad9) -> /IN1
Routing:
- net Net-(U1-CLK): track 67.3 -> 0.00 mm
- net Net-(U1-DIO): track 53.6 -> 0.00 mm
- net Net-(U1-CS): track 51.2 -> 0.00 mm
- net GND: vias 0 -> 3
Other:
- board size 178.5 x 99.4 mm -> 178.5 x 100.4 mm

Commit message: GP1294...
Parts:
- removed FILLAMENT0: MA04-1, VFD-Power:MA04-1
- moved R5 102.3 mm to (229.2, 63.8), turned to -90 degrees
- moved IC2 97.4 mm to (157.0, 59.3), turned to 0 degrees
- moved L2 96.2 mm to (192.2, 87.0), turned to -90 degrees
- moved R4 93.9 mm to (201.1, 73.5)
- moved IC3 90.9 mm to (206.2, 68.0), turned to -90 degrees
- moved IC1 88.5 mm to (192.7, 70.2), turned to -90 degrees
- moved C8 88.2 mm to (205.9, 86.8), turned to 180 degrees
- moved L3 86.4 mm to (157.0, 76.8), turned to 180 degrees
- moved C1 84.0 mm to (183.2, 61.0), turned to 180 degrees
- moved R1 83.0 mm to (183.2, 63.8), turned to 180 degrees
- moved U2 78.0 mm to (162.2, 51.5), turned to 0 degrees
- moved C4 77.8 mm to (169.8, 87.2), turned to 180 degrees
- moved U3 70.7 mm to (155.0, 103.3)
- moved D1 69.2 mm to (181.2, 87.0)
- moved L1 63.4 mm to (192.5, 81.2), turned to 0 degrees
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
Commit message: GP1294 more progress...
Parts:
- removed C6: CPOL-EU153CLV-0807, VFD-Power:153CLV-0807
- U2: footprint VFDs-Library:Teensy4.0 -> VFDs-Library:Teensy4.0_smd
- moved C2 119.4 mm to (196.5, 56.4), turned to 180 degrees
- moved C5 98.8 mm to (170.7, 100.1)
- moved C3 92.9 mm to (132.6, 142.0), turned to -90 degrees
- moved IC2 78.3 mm to (231.1, 84.6)
- moved L3 78.0 mm to (230.9, 101.9)
- moved D2 50.1 mm to (206.8, 79.5), turned to 0 degrees
- moved C4 39.7 mm to (206.8, 72.9)
- moved R6 34.9 mm to (167.9, 89.1), turned to 90 degrees
- moved R7 33.9 mm to (170.4, 89.1), turned to 90 degrees
- moved R8 33.2 mm to (172.9, 89.1), turned to 90 degrees
- moved R9 32.9 mm to (175.5, 89.1), turned to 90 degrees
- moved D1 16.7 mm to (196.3, 79.8), turned to 0 degrees
- moved U3 14.6 mm to (169.4, 105.4)
- moved C8 10.8 mm to (206.8, 97.5)
- moved L2 10.1 mm to (196.3, 96.3)
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Other:
- board size 178.5 x 100.4 mm -> 178.5 x 99.9 mm
