File: PCB-KiCad/GP1294-Teens4.kicad_sch (KiCad schematic)
At the start: 6 parts, among them SW1 RotaryEncoder_Switch, SW2 RotaryEncoder_Switch, SW3 SW_Push, SW4 SW_Push

Commit message: Progress on GP1294 board..
Parts:
- removed SW1, SW2: RotaryEncoder_Switch, Rotary_Encoder:RotaryEncoder_Alps_EC12E_Vertical_H20mm, symbol Device:RotaryEncoder_Switch
- added SW1: SW_Push, Button_Switch_THT:SW_PUSH-12mm_Wuerth-430476085716, symbol Switch:SW_Push
- added SW5, SW6: RotaryEncoder_Switch, Rotary_Encoder:RotaryEncoder_Alps_EC12E-Switch_Vertical_H20mm, symbol Device:RotaryEncoder_Switch
Connections:
- net GND: now also SW1.1
- net at U2.7 (5): now also SW1.2
Changed lines of the file:
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@@
   (junction (at 246.38 64.77) (diameter 0) (color 0 0 0 0)
   )
+  (junction (at 107.95 99.06) (diameter 0) (color 0 0 0 0)
+  )
   (junction (at 246.38 100.33) (diameter 0) (color 0 0 0 0)
   )
@@
     (stroke (width 0) (type default))
   )
+  (wire (pts (xy 107.95 99.06) (xy 107.95 106.68))
+    (stroke (width 0) (type default))
+  )
   (wire (pts (xy 246.38 118.11) (xy 246.38 120.65))
     (stroke (width 0) (type default))
@@
     (stroke (width 0) (type default))
   )
+  (wire (pts (xy 120.65 95.25) (xy 137.16 95.25))
+    (stroke (width 0) (type default))
+  )
   (wire (pts (xy 158.75 113.03) (xy 184.15 113.03))
     (stroke (width 0) (type default))
@@
     (stroke (width 0) (type default))
   )
+  (wire (pts (xy 118.11 106.68) (xy 120.65 106.68))
+    (stroke (width 0) (type default))
+  )
+  (wire (pts (xy 120.65 106.68) (xy 120.65 95.25))
+    (stroke (width 0) (type default))
+  )
   (wire (pts (xy 250.19 67.31) (xy 243.84 67.31))
     (stroke (width 0) (type default))
@@
     (stroke (width 0) (type default))
   )
+  (symbol (lib_id "Device:RotaryEncoder_Switch") (at 85.09 82.55 0) (unit 1)
+    (in_bom yes) (on_board yes) (dnp no) (fields_autoplaced)
+    (property "Reference" "SW6" (at 85.09 72.39 0)
+      (effects (font (size 1.27 1.27)))
+    )
+    (property "Value" "RotaryEncoder_Switch" (at 85.09 74.93 0)
+      (effects (font (size 1.27 1.27)))
+    )
+    (property "Footprint" "Rotary_Encoder:RotaryEncoder_Alps_EC12E-Switch_Vertical_H20mm" (at 81.28 78.486 0)
+      (effects (font (size 1.27 1.27)) hide)
+    )
+    (property "Datasheet" "~" (at 85.09 75.946 0)
+      (effects (font (size 1.27 1.27)) hide)
+    )
+    (pin "A")
+    (pin "C")
+    (pin "S1")
+    (pin "S2")
+    (pin "B")
+    (instances
+      (project "GP1294-Teens4"
+        (path "/3de011e3-f89b-42a8-8637-1f4c3f0867fa"
+          (reference "SW6") (unit 1)
+        )
+      )
+    )
+  )
   (symbol (lib_id "power:+3.3V") (at 163.83 74.93 0) (unit 1)
     (in_bom yes) (on_board yes) (dnp no) (fields_autoplaced)
@@
         (path "/3de011e3-f89b-42a8-8637-1f4c3f0867fa"
           (reference "#PWR03") (unit 1)
-        )
-      )
-    )
-  )
-  (symbol (lib_id "Device:RotaryEncoder_Switch") (at 59.69 83.82 0) (unit 1)
-    (in_bom yes) (on_board yes) (dnp no) (fields_autoplaced)
-    (property "Reference" "SW2" (at 59.69 73.66 0)
-      (effects (font (size 1.27 1.27)))
-    )
-    (property "Value" "RotaryEncoder_Switch" (at 59.69 76.2 0)
-      (effects (font (size 1.27 1.27)))
-    )
-    (property "Footprint" "Rotary_Encoder:RotaryEncoder_Alps_EC12E_Vertical_H20mm" (at 55.88 79.756 0)
-      (effects (font (size 1.27 1.27)) hide)
-    )
-    (property "Datasheet" "~" (at 59.69 77.216 0)
-      (effects (font (size 1.27 1.27)) hide)
-    )
-    (pin "C")
-    (pin "B")
-    (pin "S1")
-    (pin "A")
-    (pin "S2")
-    (instances
-      (project "GP1294-Teens4"
-        (path "/3de011e3-f89b-42a8-8637-1f4c3f0867fa"
-          (reference "SW2") (unit 1)
         )
       )
@@
     )
   )
-  (symbol (lib_id "Device:RotaryEncoder_Switch") (at 59.69 60.96 0) (unit 1)
-    (in_bom yes) (on_board yes) (dnp no) (fields_autoplaced)
-    (property "Reference" "SW1" (at 59.69 50.8 0)
-      (effects (font (size 1.27 1.27)))
-    )
-    (property "Value" "RotaryEncoder_Switch" (at 59.69 53.34 0)
-      (effects (font (size 1.27 1.27)))
-    )
-    (property "Footprint" "Rotary_Encoder:RotaryEncoder_Alps_EC12E_Vertical_H20mm" (at 55.88 56.896 0)
-      (effects (font (size 1.27 1.27)) hide)
-    )
-    (property "Datasheet" "~" (at 59.69 54.356 0)
-      (effects (font (size 1.27 1.27)) hide)
-    )
+  (symbol (lib_id "Device:RotaryEncoder_Switch") (at 85.09 60.96 0) (unit 1)
+    (in_bom yes) (on_board yes) (dnp no) (fields_autoplaced)
+    (property "Reference" "SW5" (at 85.09 50.8 0)
+      (effects (font (size 1.27 1.27)))
+    )
+    (property "Value" "RotaryEncoder_Switch" (at 85.09 53.34 0)
+      (effects (font (size 1.27 1.27)))
+    )
+    (property "Footprint" "Rotary_Encoder:RotaryEncoder_Alps_EC12E-Switch_Vertical_H20mm" (at 81.28 56.896 0)
+      (effects (font (size 1.27 1.27)) hide)
+    )
+    (property "Datasheet" "~" (at 85.09 54.356 0)
+      (effects (font (size 1.27 1.27)) hide)
+    )
+    (pin "A")
+    (pin "C")
+    (pin "S1")
     (pin "S2")
     (pin "B")
-    (pin "S1")
-    (pin "C")
-    (pin "A")
-    (instances
-      (project "GP1294-Teens4"
-        (path "/3de011e3-f89b-42a8-8637-1f4c3f0867fa"
-          (reference "SW1") (unit 1)
+    (instances
+      (project "GP1294-Teens4"
+        (path "/3de011e3-f89b-42a8-8637-1f4c3f0867fa"
+          (reference "SW5") (unit 1)
         )
       )
@@
         )
       )
+    )
+  )
+  (symbol (lib_id "Switch:SW_Push") (at 113.03 106.68 0) (unit 1)
+    (in_bom yes) (on_board yes) (dnp no) (fields_autoplaced)
+    (property "Reference" "SW1" (at 113.03 99.06 0)
+      (effects (font (size 1.27 1.27)))
+    )
+    (property "Value" "SW_Push" (at 113.03 101.6 0)
+      (effects (font (size 1.27 1.27)))
+    )
+    (property "Footprint" "Button_Switch_THT:SW_PUSH-12mm_Wuerth-430476085716" (at 113.03 101.6 0)
+      (effects (font (size 1.27 1.27)) hide)
+    )
+    (property "Datasheet" "~" (at 113.03 101.6 0)
+      (effects (font (size 1.27 1.27)) hide)
+    )
+    (pin "1")
+    (pin "2")
+    (instances
+      (project "GP1294-Teens4"
+        (path "/3de011e3-f89b-42a8-8637-1f4c3f0867fa"
+          (reference "SW1") (unit 1)
+        )
+      )

Commit message: GP1294 progress..
Parts:
- added Case1: ~, VFDs-Library:CaseDD, symbol VFDs-Library:CaseDD
- added SW2, SW5: SW_Push, Button_Switch_THT:SW_PUSH-12mm_Wuerth-430476085716, symbol Switch:SW_Push
- renumbered SW5 to ENC1, SW6 to ENC2
Changed lines of the file:
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@@
   (symbol (lib_id "Device:RotaryEncoder_Switch") (at 85.09 82.55 0) (unit 1)
     (in_bom yes) (on_board yes) (dnp no) (fields_autoplaced)
-    (property "Reference" "SW6" (at 85.09 72.39 0)
+    (property "Reference" "ENC2" (at 85.09 72.39 0)
       (effects (font (size 1.27 1.27)))
     )
@@
     )
     (pin "A")
+    (pin "B")
     (pin "C")
     (pin "S1")
     (pin "S2")
-    (pin "B")
-    (instances
-      (project "GP1294-Teens4"
-        (path "/3de011e3-f89b-42a8-8637-1f4c3f0867fa"
-          (reference "SW6") (unit 1)
+    (instances
+      (project "GP1294-Teens4"
+        (path "/3de011e3-f89b-42a8-8637-1f4c3f0867fa"
+          (reference "ENC2") (unit 1)
         )
       )
@@
     )
   )
+  (symbol (lib_id "Switch:SW_Push") (at 114.935 118.11 0) (unit 1)
+    (in_bom yes) (on_board yes) (dnp no) (fields_autoplaced)
+    (property "Reference" "SW2" (at 114.935 110.49 0)
+      (effects (font (size 1.27 1.27)))
+    )
+    (property "Value" "SW_Push" (at 114.935 113.03 0)
+      (effects (font (size 1.27 1.27)))
+    )
+    (property "Footprint" "Button_Switch_THT:SW_PUSH-12mm_Wuerth-430476085716" (at 114.935 113.03 0)
+      (effects (font (size 1.27 1.27)) hide)
+    )
+    (property "Datasheet" "~" (at 114.935 113.03 0)
+      (effects (font (size 1.27 1.27)) hide)
+    )
+    (pin "1")
+    (pin "2")
+    (instances
+      (project "GP1294-Teens4"
+        (path "/3de011e3-f89b-42a8-8637-1f4c3f0867fa"
+          (reference "SW2") (unit 1)
+        )
+      )
+    )
+  )
   (symbol (lib_id "power:GND") (at 171.45 82.55 0) (unit 1)
     (in_bom yes) (on_board yes) (dnp no) (fields_autoplaced)
@@
         (path "/3de011e3-f89b-42a8-8637-1f4c3f0867fa"
           (reference "#PWR06") (unit 1)
+        )
+      )
+    )
+  )
+  (symbol (lib_id "Switch:SW_Push") (at 114.935 128.905 0) (unit 1)
+    (in_bom yes) (on_board yes) (dnp no) (fields_autoplaced)
+    (property "Reference" "SW5" (at 114.935 121.285 0)
+      (effects (font (size 1.27 1.27)))
+    )
+    (property "Value" "SW_Push" (at 114.935 123.825 0)
+      (effects (font (size 1.27 1.27)))
+    )
+    (property "Footprint" "Button_Switch_THT:SW_PUSH-12mm_Wuerth-430476085716" (at 114.935 123.825 0)
+      (effects (font (size 1.27 1.27)) hide)
+    )
+    (property "Datasheet" "~" (at 114.935 123.825 0)
+      (effects (font (size 1.27 1.27)) hide)
+    )
+    (pin "1")
+    (pin "2")
+    (instances
+      (project "GP1294-Teens4"
+        (path "/3de011e3-f89b-42a8-8637-1f4c3f0867fa"
+          (reference "SW5") (unit 1)
         )
       )
@@
       (effects (font (size 1.27 1.27)) hide)
     )
-    (pin "7")
-    (pin "6")
+    (pin "1")
+    (pin "10")
+    (pin "11")
+    (pin "12")
+    (pin "13")
+    (pin "14")
+    (pin "15")
+    (pin "16")
+    (pin "17")
+    (pin "18")
+    (pin "19")
+    (pin "2")
+    (pin "20")
+    (pin "21")
+    (pin "22")
+    (pin "23")
+    (pin "24")
+    (pin "25")
+    (pin "26")
+    (pin "27")
+    (pin "28")
+    (pin "29")
+    (pin "3")
     (pin "30")
+    (pin "31")
     (pin "4")
     (pin "5")
-    (pin "29")
-    (pin "23")
-    (pin "28")
-    (pin "25")
-    (pin "24")
-    (pin "1")
-    (pin "10")
-    (pin "26")
-    (pin "3")
-    (pin "22")
-    (pin "21")
-    (pin "20")
-    (pin "15")
-    (pin "16")
-    (pin "27")
-    (pin "31")
-    (pin "2")
-    (pin "12")
-    (pin "14")
-    (pin "17")
-    (pin "13")
-    (pin "18")
-    (pin "19")
+    (pin "6")
+    (pin "7")
     (pin "8")
     (pin "9")
-    (pin "11")
     (instances
       (project "GP1294-Teens4"
@@
   (symbol (lib_id "Device:RotaryEncoder_Switch") (at 85.09 60.96 0) (unit 1)
     (in_bom yes) (on_board yes) (dnp no) (fields_autoplaced)
-    (property "Reference" "SW5" (at 85.09 50.8 0)
+    (property "Reference" "ENC1" (at 85.09 50.8 0)
       (effects (font (size 1.27 1.27)))
     )
@@
     )
     (pin "A")
+    (pin "B")
     (pin "C")
     (pin "S1")
     (pin "S2")
-    (pin "B")
-    (instances
-      (project "GP1294-Teens4"
-        (path "/3de011e3-f89b-42a8-8637-1f4c3f0867fa"
-          (reference "SW5") (unit 1)
+    (instances
+      (project "GP1294-Teens4"
+        (path "/3de011e3-f89b-42a8-8637-1f4c3f0867fa"
+          (reference "ENC1") (unit 1)
         )
       )
@@
       (effects (font (size 1.27 1.27)) hide)
     )
+    (pin "1")
+    (pin "10")
+    (pin "11")
+    (pin "12")
+    (pin "13")
+    (pin "14")
+    (pin "15")
     (pin "16")
-    (pin "10")
     (pin "17")
-    (pin "1")
+    (pin "18")
+    (pin "19")
+    (pin "2")
+    (pin "20")
+    (pin "21")
+    (pin "22")
+    (pin "23")
+    (pin "24")
     (pin "25")
-    (pin "5")
+    (pin "26")
+    (pin "27")
+    (pin "28")
     (pin "3")
     (pin "4")
-    (pin "27")
-    (pin "26")
-    (pin "21")
-    (pin "22")
+    (pin "5")
+    (pin "6")
+    (pin "7")
+    (pin "8")
     (pin "9")
-    (pin "23")
-    (pin "24")
-    (pin "28")
-    (pin "6")
-    (pin "8")
-    (pin "7")
-    (pin "15")
-    (pin "12")
-    (pin "19")
-    (pin "2")
-    (pin "13")
-    (pin "14")
-    (pin "11")
-    (pin "18")
-    (pin "20")
     (instances
       (project "GP1294-Teens4"
@@
         )
       )
+    )
+  )
+  (symbol (lib_id "VFDs-Library:CaseDD") (at 31.75 31.115 0) (unit 1)
+    (in_bom yes) (on_board yes) (dnp no) (fields_autoplaced)
+    (property "Reference" "Case1" (at 34.29 31.75 0)
+      (effects (font (size 1.27 1.27)) (justify left))
+    )
+    (property "Value" "~" (at 31.75 31.115 0)
+      (effects (font (size 1.27 1.27)))
+    )
+    (property "Footprint" "VFDs-Library:CaseDD" (at 31.75 31.115 0)
+      (effects (font (size 1.27 1.27)) hide)
+    )
+    (property "Datasheet" "" (at 31.75 31.115 0)
+      (effects (font (size 1.27 1.27)) hide)
+    )
+    (instances
+      (project "GP1294-Teens4"
+        (path "/3de011e3-f89b-42a8-8637-1f4c3f0867fa"
+          (reference "Case1") (unit 1)
+        )
+      )

Commit message: GP1294 progress...
Parts:
- added R6, R7, R8, R9: 100, Resistor_SMD:R_0603_1608Metric, symbol Device:R
- added U4: ~, FreeDSP:FreeDSP-allinone, symbol FreeDSP:FreeDSP-allinone
Connections:
- net +24V: now also U4.1 (V+)
- net GND: now also U4.10 (GND), U4.12 (GND), U4.14 (GND), U4.16 (GND), U4.2 (GND), U4.4 (GND), U4.6 (GND), U4.8 (GND)
- net F1: now reaches U1.1 (F+)
- net F2: now reaches U1.28 (F-)
- net LRCLK1: now reaches U2.20 (A4)
- net LRCLK1: now also R9.1
- net BCLK1: now reaches U2.21 (A5)
- net BCLK1: now also R8.1
- net OUT1: now reaches U2.8 (6)
- net OUT1: now also R6.1
- net IN1: now reaches U2.9 (7)
- net IN1: now also R7.1
- new net: R6.2, U4.3 (MP1/MDI)
- new net: R7.2, U4.5 (MP8/MDO)
- new net: R8.2, U4.7 (MP11/BCLK)
- new net: R9.2, U4.9 (MP10/LRCLK)

Commit message: GP1294 more progress...
Parts:
- U2: footprint VFDs-Library:Teensy4.0 -> VFDs-Library:Teensy4.0_smd
Changed lines of the file:
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@@
       (effects (font (size 1.27 1.27)))
     )
-    (property "Footprint" "VFDs-Library:Teensy4.0" (at 135.3412 69.7725 0)
+    (property "Footprint" "VFDs-Library:Teensy4.0_smd" (at 135.3412 69.7725 0)
       (effects (font (size 1.27 1.27)) hide)
     )

Commit message: GP12.. better case and stuff
Parts:
- removed ENC1, ENC2: RotaryEncoder_Switch, Rotary_Encoder:RotaryEncoder_Alps_EC12E-Switch_Vertical_H20mm, symbol Device:RotaryEncoder_Switch
- removed SW1, SW2, SW3, SW4, SW5: SW_Push, Button_Switch_THT:SW_PUSH-12mm_Wuerth-430476085716, symbol Switch:SW_Push
- added R11, R12: 10k, Resistor_SMD:R_0603_1608Metric, symbol Device:R
Connections:
- net +3.3V: now also R11.1, R12.1
- net SDA: now reaches U4.11 (SDA)
- net SDA: now also U2.18 (A2), R12.2
- net SCL: now reaches U4.13 (SCL)
- net SCL: now also U2.19 (A3), R11.2
Other:
- added sheet inputs (inputs.kicad_sch)
