File: PCB-KiCad/VFD-Power.kicad_sch (KiCad schematic)
At the start: 25 parts, among them IC1 74132D, IC2 XL6009, IC3 ZXBM5210, U3 R-78B5.0-2.0

Commit message: GP1294 progress...
Parts:
- removed POWER0: MA06-1, VFD-Power:MA06-1, symbol VFD-Power-eagle-import:MA06-1
Changed lines of the file:
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@@
   (junction (at 161.29 53.34) (diameter 0) (color 0 0 0 0)
   )
+  (junction (at 254 45.72) (diameter 0) (color 0 0 0 0)
+  )
   (junction (at 163.83 53.34) (diameter 0) (color 0 0 0 0)
   )
@@
   (junction (at 29.21 154.94) (diameter 0) (color 0 0 0 0)
   )
-  (junction (at 33.02 48.26) (diameter 0) (color 0 0 0 0)
+  (junction (at 256.54 43.18) (diameter 0) (color 0 0 0 0)
   )
   (junction (at 179.07 78.74) (diameter 0) (color 0 0 0 0)
@@
     (stroke (width 0.1524) (type solid))
   )
+  (wire (pts (xy 255.27 49.53) (xy 254 49.53))
+    (stroke (width 0) (type default))
+  )
   (wire (pts (xy 224.79 55.88) (xy 224.79 66.04))
     (stroke (width 0.1524) (type solid))
@@
     (stroke (width 0.1524) (type solid))
   )
+  (wire (pts (xy 254 45.72) (xy 204.47 45.72))
+    (stroke (width 0) (type default))
+  )
   (wire (pts (xy 29.21 139.7) (xy 29.21 143.51))
     (stroke (width 0.1524) (type solid))
@@
     (stroke (width 0) (type default))
   )
+  (wire (pts (xy 254 49.53) (xy 254 45.72))
+    (stroke (width 0) (type default))
+  )
   (wire (pts (xy 163.83 19.05) (xy 163.83 53.34))
     (stroke (width 0) (type default))
@@
     (stroke (width 0.1524) (type solid))
   )
+  (wire (pts (xy 256.54 40.64) (xy 256.54 43.18))
+    (stroke (width 0) (type default))
+  )
   (wire (pts (xy 118.11 152.4) (xy 118.11 154.94))
     (stroke (width 0.1524) (type solid))
@@
     (stroke (width 0.1524) (type solid))
   )
-  (wire (pts (xy 266.7 43.18) (xy 212.09 43.18))
+  (wire (pts (xy 266.7 43.18) (xy 256.54 43.18))
     (stroke (width 0) (type default))
   )
@@
     (stroke (width 0.1524) (type solid))
   )
+  (wire (pts (xy 130.81 53.34) (xy 137.16 53.34))
+    (stroke (width 0) (type default))
+  )
+  (wire (pts (xy 29.21 154.94) (xy 24.13 154.94))
+    (stroke (width 0.1524) (type solid))
+  )
+  (wire (pts (xy 33.02 43.18) (xy 33.02 41.91))
+    (stroke (width 0.1524) (type solid))
+  )
+  (wire (pts (xy 118.11 162.56) (xy 110.49 162.56))
+    (stroke (width 0.1524) (type solid))
+  )
+  (wire (pts (xy 105.41 162.56) (xy 110.49 162.56))
+    (stroke (width 0.1524) (type solid))
+  )
+  (wire (pts (xy 29.21 121.92) (xy 29.21 139.7))
+    (stroke (width 0.1524) (type solid))
+  )
+  (wire (pts (xy 173.99 53.34) (xy 179.07 53.34))
+    (stroke (width 0.1524) (type solid))
+  )
+  (wire (pts (xy 191.77 91.44) (xy 191.77 93.98))
+    (stroke (width 0.1524) (type solid))
+  )
+  (wire (pts (xy 50.8 121.92) (xy 54.61 121.92))
+    (stroke (width 0.1524) (type solid))
+  )
+  (wire (pts (xy 115.57 147.32) (xy 118.11 147.32))
+    (stroke (width 0.1524) (type solid))
+  )
+  (wire (pts (xy 50.8 160.02) (xy 50.8 157.48))
+    (stroke (width 0.1524) (type solid))
+  )
+  (wire (pts (xy 86.36 172.72) (xy 86.36 170.18))
+    (stroke (width 0.1524) (type solid))
+  )
+  (wire (pts (xy 63.5 40.64) (xy 63.5 35.56))
+    (stroke (width 0.1524) (type solid))
+  )
+  (wire (pts (xy 41.91 35.56) (xy 46.99 35.56))
+    (stroke (width 0.1524) (type solid))
+  )
+  (wire (pts (xy 78.74 147.32) (xy 86.36 147.32))
+    (stroke (width 0.1524) (type solid))
+  )
+  (wire (pts (xy 189.23 45.72) (xy 189.23 53.34))
+    (stroke (width 0.1524) (type solid))
+  )
+  (wire (pts (xy 196.85 50.8) (xy 196.85 40.64))
+    (stroke (width 0.1524) (type solid))
+  )
   (wire (pts (xy 33.02 48.26) (xy 41.91 48.26))
-    (stroke (width 0) (type default))
-  )
-  (wire (pts (xy 130.81 53.34) (xy 137.16 53.34))
-    (stroke (width 0) (type default))
-  )
-  (wire (pts (xy 29.21 154.94) (xy 24.13 154.94))
-    (stroke (width 0.1524) (type solid))
-  )
-  (wire (pts (xy 33.02 43.18) (xy 33.02 41.91))
-    (stroke (width 0.1524) (type solid))
-  )
-  (wire (pts (xy 118.11 162.56) (xy 110.49 162.56))
-    (stroke (width 0.1524) (type solid))
-  )
-  (wire (pts (xy 105.41 162.56) (xy 110.49 162.56))
-    (stroke (width 0.1524) (type solid))
-  )
-  (wire (pts (xy 29.21 121.92) (xy 29.21 139.7))
-    (stroke (width 0.1524) (type solid))
-  )
-  (wire (pts (xy 173.99 53.34) (xy 179.07 53.34))
-    (stroke (width 0.1524) (type solid))
-  )
-  (wire (pts (xy 191.77 91.44) (xy 191.77 93.98))
-    (stroke (width 0.1524) (type solid))
-  )
-  (wire (pts (xy 50.8 121.92) (xy 54.61 121.92))
-    (stroke (width 0.1524) (type solid))
-  )
-  (wire (pts (xy 115.57 147.32) (xy 118.11 147.32))
-    (stroke (width 0.1524) (type solid))
-  )
-  (wire (pts (xy 50.8 160.02) (xy 50.8 157.48))
-    (stroke (width 0.1524) (type solid))
-  )
-  (wire (pts (xy 86.36 172.72) (xy 86.36 170.18))
-    (stroke (width 0.1524) (type solid))
-  )
-  (wire (pts (xy 63.5 40.64) (xy 63.5 35.56))
-    (stroke (width 0.1524) (type solid))
-  )
-  (wire (pts (xy 41.91 35.56) (xy 46.99 35.56))
-    (stroke (width 0.1524) (type solid))
-  )
-  (wire (pts (xy 78.74 147.32) (xy 86.36 147.32))
-    (stroke (width 0.1524) (type solid))
-  )
-  (wire (pts (xy 189.23 45.72) (xy 189.23 53.34))
-    (stroke (width 0.1524) (type solid))
-  )
-  (wire (pts (xy 196.85 50.8) (xy 196.85 40.64))
-    (stroke (width 0.1524) (type solid))
-  )
-  (wire (pts (xy 33.02 48.26) (xy 41.91 48.26))
     (stroke (width 0.1524) (type solid))
   )
@@
     (stroke (width 0.1524) (type solid))
   )
-  (wire (pts (xy 266.7 45.72) (xy 204.47 45.72))
+  (wire (pts (xy 266.7 45.72) (xy 254 45.72))
     (stroke (width 0) (type default))
   )
@@
   (wire (pts (xy 69.85 147.32) (xy 73.66 147.32))
     (stroke (width 0.1524) (type solid))
+  )
+  (wire (pts (xy 256.54 43.18) (xy 212.09 43.18))
+    (stroke (width 0) (type default))
   )
   (wire (pts (xy 46.99 35.56) (xy 54.61 35.56))
@@
     (effects (font (size 1.2446 1.2446)) (justify left bottom))
   )
+  (global_label "F1" (shape input) (at 255.27 49.53 0) (fields_autoplaced)
+    (effects (font (size 1.27 1.27)) (justify left))
+    (property "Intersheetrefs" "${INTERSHEET_REFS}" (at 260.5533 49.53 0)
+      (effects (font (size 1.27 1.27)) (justify left) hide)
+    )
+  )
+  (global_label "F2" (shape input) (at 256.54 40.64 0) (fields_autoplaced)
+    (effects (font (size 1.27 1.27)) (justify left))
+    (property "Intersheetrefs" "${INTERSHEET_REFS}" (at 261.8233 40.64 0)
+      (effects (font (size 1.27 1.27)) (justify left) hide)
+    )
+  )
   (hierarchical_label "VPP" (shape output) (at 267.97 134.62 0) (fields_autoplaced)
     (effects (font (size 3 3)) (justify left))
@@
   (hierarchical_label "F1" (shape output) (at 266.7 52.07 0) (fields_autoplaced)
     (effects (font (size 3 3)) (justify left))
+  )
+  (hierarchical_label "V+" (shape input) (at 33.02 38.1 180) (fields_autoplaced)
+    (effects (font (size 1.27 1.27)) (justify right))
   )
   (hierarchical_label "5V" (shape output) (at 163.83 19.05 0) (fields_autoplaced)
@@
         )
       )
-    )
-  )
-  (symbol (lib_id "VFD-Power-eagle-import:MA06-1") (at 25.4 43.18 0) (unit 1)
-    (in_bom yes) (on_board yes) (dnp no)
-    (property "Reference" "POWER0" (at 24.13 34.798 0)
-      (effects (font (size 1.778 1.5113)) (justify left bottom))
-    )
-    (property "Value" "MA06-1" (at 24.13 55.88 0)
-      (effects (font (size 1.778 1.5113)) (justify left bottom) hide)
-    )
-    (property "Footprint" "VFD-Power:MA06-1" (at 25.4 43.18 0)
-      (effects (font (size 1.27 1.27)) hide)
-    )
-    (property "Datasheet" "" (at 25.4 43.18 0)
-      (effects (font (size 1.27 1.27)) hide)
-    )
-    (pin "1")
-    (pin "2")
-    (pin "3")
-    (pin "4")
-    (pin "5")
-    (pin "6")
-    (instances
-      (project "GP1294-Teens4"
-        (path "/3de011e3-f89b-42a8-8637-1f4c3f0867fa/9e049bd2-8c7e-4a7a-b856-b0fbd11ae8df"
-          (reference "POWER0") (unit 1)
-        )
-      )
-      (project "VFD-Power"
-        (path "/d66e9896-ee3f-419d-ab82-78a854ae4100"
-          (reference "POWER0") (unit 1)
-        )
-      )

Commit message: GP1294...
Parts:
- removed FILLAMENT0: MA04-1, VFD-Power:MA04-1, symbol VFD-Power-eagle-import:MA04-1
Other:
- moved on the sheet: R5
Changed lines of the file:
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@@
   (junction (at 63.5 35.56) (diameter 0) (color 0 0 0 0)
   )
-  (junction (at 212.09 40.64) (diameter 0) (color 0 0 0 0)
+  (junction (at 254 34.925) (diameter 0) (color 0 0 0 0)
+  )
+  (junction (at 255.27 42.545) (diameter 0) (color 0 0 0 0)
   )
   (junction (at 191.77 93.98) (diameter 0) (color 0 0 0 0)
@@
   (junction (at 161.29 53.34) (diameter 0) (color 0 0 0 0)
   )
-  (junction (at 254 45.72) (diameter 0) (color 0 0 0 0)
-  )
   (junction (at 163.83 53.34) (diameter 0) (color 0 0 0 0)
   )
@@
   (junction (at 46.99 35.56) (diameter 0) (color 0 0 0 0)
   )
-  (junction (at 204.47 40.64) (diameter 0) (color 0 0 0 0)
-  )
   (junction (at 217.17 93.98) (diameter 0) (color 0 0 0 0)
   )
@@
   (junction (at 29.21 154.94) (diameter 0) (color 0 0 0 0)
   )
-  (junction (at 256.54 43.18) (diameter 0) (color 0 0 0 0)
-  )
   (junction (at 179.07 78.74) (diameter 0) (color 0 0 0 0)
   )
@@
     (stroke (width 0.1524) (type solid))
   )
-  (wire (pts (xy 255.27 49.53) (xy 254 49.53))
+  (wire (pts (xy 254.635 31.75) (xy 254 31.75))
     (stroke (width 0) (type default))
   )
@@
     (stroke (width 0) (type default))
   )
-  (wire (pts (xy 204.47 40.64) (xy 207.01 40.64))
-    (stroke (width 0.1524) (type solid))
-  )
   (wire (pts (xy 196.85 73.66) (xy 189.23 78.74))
     (stroke (width 0.1524) (type solid))
@@
     (stroke (width 0.1524) (type solid))
   )
-  (wire (pts (xy 234.95 40.64) (xy 234.95 53.34))
+  (wire (pts (xy 224.79 42.545) (xy 224.79 53.34))
     (stroke (width 0.1524) (type solid))
   )
@@
     (stroke (width 0.1524) (type solid))
   )
-  (wire (pts (xy 254 45.72) (xy 204.47 45.72))
+  (wire (pts (xy 254 34.925) (xy 196.85 34.925))
     (stroke (width 0) (type default))
   )
@@
     (stroke (width 0.1524) (type solid))
   )
+  (wire (pts (xy 196.85 34.925) (xy 196.85 50.8))
+    (stroke (width 0) (type default))
+  )
   (wire (pts (xy 196.85 58.42) (xy 196.85 63.5))
     (stroke (width 0.1524) (type solid))
@@
     (stroke (width 0.1524) (type solid))
   )
+  (wire (pts (xy 255.27 42.545) (xy 264.16 42.545))
+    (stroke (width 0) (type default))
+  )
   (wire (pts (xy 105.41 147.32) (xy 105.41 152.4))
     (stroke (width 0.1524) (type solid))
@@
     (stroke (width 0) (type default))
   )
-  (wire (pts (xy 254 49.53) (xy 254 45.72))
-    (stroke (width 0) (type default))
-  )
   (wire (pts (xy 163.83 19.05) (xy 163.83 53.34))
     (stroke (width 0) (type default))
@@
     (stroke (width 0) (type default))
   )
+  (wire (pts (xy 255.27 38.735) (xy 255.27 42.545))
+    (stroke (width 0) (type default))
+  )
   (wire (pts (xy 29.21 154.94) (xy 29.21 151.13))
     (stroke (width 0.1524) (type solid))
@@
     (stroke (width 0.1524) (type solid))
   )
-  (wire (pts (xy 256.54 40.64) (xy 256.54 43.18))
+  (wire (pts (xy 254 31.75) (xy 254 34.925))
     (stroke (width 0) (type default))
   )
@@
     (stroke (width 0.1524) (type solid))
   )
-  (wire (pts (xy 234.95 53.34) (xy 222.25 53.34))
+  (wire (pts (xy 224.79 53.34) (xy 222.25 53.34))
     (stroke (width 0.1524) (type solid))
   )
@@
     (stroke (width 0.1524) (type solid))
   )
-  (wire (pts (xy 212.09 43.18) (xy 212.09 40.64))
-    (stroke (width 0) (type default))
-  )
   (wire (pts (xy 58.42 147.32) (xy 69.85 147.32))
     (stroke (width 0.1524) (type solid))
@@
     (stroke (width 0.1524) (type solid))
   )
-  (wire (pts (xy 266.7 43.18) (xy 256.54 43.18))
-    (stroke (width 0) (type default))
-  )
   (wire (pts (xy 29.21 139.7) (xy 24.13 139.7))
     (stroke (width 0.1524) (type solid))
@@
     (stroke (width 0.1524) (type solid))
   )
-  (wire (pts (xy 196.85 50.8) (xy 196.85 40.64))
-    (stroke (width 0.1524) (type solid))
+  (wire (pts (xy 234.95 42.545) (xy 255.27 42.545))
+    (stroke (width 0) (type default))
   )
   (wire (pts (xy 33.02 48.26) (xy 41.91 48.26))
@@
     (stroke (width 0.1524) (type solid))
   )
-  (wire (pts (xy 266.7 45.72) (xy 254 45.72))
+  (wire (pts (xy 264.16 34.925) (xy 254 34.925))
     (stroke (width 0) (type default))
   )
@@
     (stroke (width 0.1524) (type solid))
   )
-  (wire (pts (xy 212.09 40.64) (xy 224.79 40.64))
-    (stroke (width 0.1524) (type solid))
-  )
   (wire (pts (xy 194.31 66.04) (xy 194.31 55.88))
     (stroke (width 0.1524) (type solid))
@@
     (stroke (width 0.1524) (type solid))
   )
-  (wire (pts (xy 256.54 43.18) (xy 212.09 43.18))
-    (stroke (width 0) (type default))
-  )
   (wire (pts (xy 46.99 35.56) (xy 54.61 35.56))
     (stroke (width 0.1524) (type solid))
@@
     (stroke (width 0.1524) (type solid))
   )
-  (wire (pts (xy 204.47 45.72) (xy 204.47 40.64))
-    (stroke (width 0) (type default))
-  )
-  (wire (pts (xy 266.7 45.72) (xy 266.7 52.07))
-    (stroke (width 0) (type default))
-  )
   (wire (pts (xy 217.17 93.98) (xy 214.63 93.98))
     (stroke (width 0.1524) (type solid))
@@
   )
   (wire (pts (xy 63.5 50.8) (xy 63.5 48.26))
-    (stroke (width 0.1524) (type solid))
-  )
-  (wire (pts (xy 196.85 40.64) (xy 204.47 40.64))
-    (stroke (width 0.1524) (type solid))
-  )
-  (wire (pts (xy 209.55 40.64) (xy 212.09 40.64))
     (stroke (width 0.1524) (type solid))
   )
@@
     (effects (font (size 4 4)) (justify left bottom))
   )
-  (label "F1" (at 196.85 40.64 0) (fields_autoplaced)
+  (label "F1" (at 198.12 42.545 0) (fields_autoplaced)
     (effects (font (size 1.2446 1.2446)) (justify left bottom))
   )
-  (label "F2" (at 219.71 40.64 0) (fields_autoplaced)
-    (effects (font (size 1.2446 1.2446)) (justify left bottom))
+  (label "F2" (at 223.52 43.18 180) (fields_autoplaced)
+    (effects (font (size 1.2446 1.2446)) (justify right bottom))
   )
   (label "FF_BLANK" (at 158.75 78.74 0) (fields_autoplaced)
@@
     (effects (font (size 1.2446 1.2446)) (justify left bottom))
   )
-  (global_label "F1" (shape input) (at 255.27 49.53 0) (fields_autoplaced)
+  (global_label "F1" (shape input) (at 254.635 31.75 0) (fields_autoplaced)
     (effects (font (size 1.27 1.27)) (justify left))
-    (property "Intersheetrefs" "${INTERSHEET_REFS}" (at 260.5533 49.53 0)
+    (property "Intersheetrefs" "${INTERSHEET_REFS}" (at 259.9183 31.75 0)
       (effects (font (size 1.27 1.27)) (justify left) hide)
     )
   )
-  (global_label "F2" (shape input) (at 256.54 40.64 0) (fields_autoplaced)
+  (global_label "F2" (shape input) (at 255.27 38.735 0) (fields_autoplaced)
     (effects (font (size 1.27 1.27)) (justify left))
-    (property "Intersheetrefs" "${INTERSHEET_REFS}" (at 261.8233 40.64 0)
+    (property "Intersheetrefs" "${INTERSHEET_REFS}" (at 260.5533 38.735 0)
       (effects (font (size 1.27 1.27)) (justify left) hide)
     )
@@
     (effects (font (size 3 3)) (justify left))
   )
-  (hierarchical_label "F2" (shape output) (at 266.7 43.18 0) (fields_autoplaced)
+  (hierarchical_label "F2" (shape output) (at 264.16 42.545 0) (fields_autoplaced)
     (effects (font (size 3 3)) (justify left))
   )
-  (hierarchical_label "F1" (shape output) (at 266.7 52.07 0) (fields_autoplaced)
+  (hierarchical_label "F1" (shape output) (at 264.16 34.925 0) (fields_autoplaced)
     (effects (font (size 3 3)) (justify left))
   )
@@
     )
   )
-  (symbol (lib_id "VFD-Power-eagle-import:R-EU_0411/15") (at 229.87 40.64 0) (unit 1)
-    (in_bom yes) (on_board yes) (dnp no)
-    (property "Reference" "R5" (at 226.06 39.1414 0)
-      (effects (font (size 1.778 1.5113)) (justify left bottom))
-    )
-    (property "Value" "22" (at 226.06 43.942 0)
-      (effects (font (size 1.778 1.5113)) (justify left bottom))
-    )
-    (property "Footprint" "VFD-Power:0411_15" (at 229.87 40.64 0)
-      (effects (font (size 1.27 1.27)) hide)
-    )
-    (property "Datasheet" "" (at 229.87 40.64 0)
+  (symbol (lib_id "VFD-Power-eagle-import:R-EU_0411/15") (at 229.87 42.545 180) (unit 1)
+    (in_bom yes) (on_board yes) (dnp no)
+    (property "Reference" "R5" (at 233.68 44.0436 0)
+      (effects (font (size 1.778 1.5113)) (justify left bottom))
+    )
+    (property "Value" "22" (at 233.68 39.243 0)
+      (effects (font (size 1.778 1.5113)) (justify left bottom))
+    )
+    (property "Footprint" "VFD-Power:0411_15" (at 229.87 42.545 0)
+      (effects (font (size 1.27 1.27)) hide)
+    )
+    (property "Datasheet" "" (at 229.87 42.545 0)
       (effects (font (size 1.27 1.27)) hide)
     )
@@
         )
       )
-    )
-  )
-  (symbol (lib_id "VFD-Power-eagle-import:MA04-1") (at 209.55 33.02 270) (unit 1)
-    (in_bom yes) (on_board yes) (dnp no)
-    (property "Reference" "FILLAMENT0" (at 215.392 31.75 0)
-      (effects (font (size 1.778 1.5113)) (justify left bottom))
-    )
-    (property "Value" "MA04-1" (at 199.39 31.75 0)
-      (effects (font (size 1.778 1.5113)) (justify left bottom) hide)
-    )
-    (property "Footprint" "VFD-Power:MA04-1" (at 209.55 33.02 0)
-      (effects (font (size 1.27 1.27)) hide)
-    )
-    (property "Datasheet" "" (at 209.55 33.02 0)
-      (effects (font (size 1.27 1.27)) hide)
-    )
-    (pin "1")
-    (pin "2")
-    (pin "3")
-    (pin "4")
-    (instances
-      (project "GP1294-Teens4"
-        (path "/3de011e3-f89b-42a8-8637-1f4c3f0867fa/9e049bd2-8c7e-4a7a-b856-b0fbd11ae8df"
-          (reference "FILLAMENT0") (unit 1)
-        )
-      )
-      (project "VFD-Power"
-        (path "/d66e9896-ee3f-419d-ab82-78a854ae4100"
-          (reference "FILLAMENT0") (unit 1)
-        )
-      )

Commit message: GP1294 more progress...
Parts:
- removed C6: CPOL-EU153CLV-0807, VFD-Power:153CLV-0807, symbol VFD-Power-eagle-import:CPOL-EU153CLV-0807
Changed lines of the file:
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@@
-    )
-  )
-  (symbol (lib_id "VFD-Power-eagle-import:CPOL-EU153CLV-0807") (at 29.21 146.05 0) (unit 1)
-    (in_bom yes) (on_board yes) (dnp no)
-    (property "Reference" "C6" (at 30.353 145.5674 0)
-      (effects (font (size 1.778 1.5113)) (justify left bottom))
-    )
-    (property "Value" "CPOL-EU153CLV-0807" (at 30.353 150.6474 0)
-      (effects (font (size 1.778 1.5113)) (justify left bottom) hide)
-    )
-    (property "Footprint" "VFD-Power:153CLV-0807" (at 29.21 146.05 0)
-      (effects (font (size 1.27 1.27)) hide)
-    )
-    (property "Datasheet" "" (at 29.21 146.05 0)
-      (effects (font (size 1.27 1.27)) hide)
-    )
-    (pin "+")
-    (pin "-")
-    (instances
-      (project "GP1294-Teens4"
-        (path "/3de011e3-f89b-42a8-8637-1f4c3f0867fa/9e049bd2-8c7e-4a7a-b856-b0fbd11ae8df"
-          (reference "C6") (unit 1)
-        )
-      )
-      (project "VFD-Power"
-        (path "/d66e9896-ee3f-419d-ab82-78a854ae4100"
-          (reference "C6") (unit 1)
-        )
-      )
     )
   )
