File: PCB-KiCad/inputs.kicad_sch (KiCad schematic)
At the start: 39 parts, among them SW1 SW_DPDT_x2, SW2 SW_DPDT_x2, SW3 SW_DPDT_x2, SW4 SW_DPDT_x2, SW5 SW_DPDT_x2, U5 ATtiny84A-P, U6 74HC165, U7 74HC165

Commit message: Checks and Firmware after 1st build.
Parts:
- R10: value 100 -> 4.7k
Changed lines of the file:
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@@
       (effects (font (size 1.27 1.27)) hide)
     )
-    (pin "2")
-    (pin "1")
+    (pin "1")
+    (pin "2")
     (instances
       (project "GP1294-Teens4"
@@
       (effects (font (size 1.27 1.27)) hide)
     )
-    (pin "2")
-    (pin "1")
+    (pin "1")
+    (pin "2")
     (instances
       (project "GP1294-Teens4"
@@
       (effects (font (size 1.27 1.27)))
     )
-    (property "Value" "100" (at 186.69 128.27 90)
+    (property "Value" "4.7k" (at 186.69 128.27 90)
       (effects (font (size 1.27 1.27)))
     )
@@
       (effects (font (size 1.27 1.27)) hide)
     )
-    (pin "2")
-    (pin "1")
+    (pin "1")
+    (pin "2")
     (instances
       (project "GP1294-Teens4"
@@
       (effects (font (size 1.27 1.27)) hide)
     )
-    (pin "2")
-    (pin "1")
+    (pin "1")
+    (pin "2")
     (instances
       (project "GP1294-Teens4"
@@
       (effects (font (size 1.27 1.27)) hide)
     )
-    (pin "2")
-    (pin "1")
+    (pin "1")
+    (pin "2")
     (instances
       (project "GP1294-Teens4"
@@
       (effects (font (size 1.27 1.27)) hide)
     )
-    (pin "2")
-    (pin "1")
+    (pin "1")
+    (pin "2")
     (instances
       (project "GP1294-Teens4"
@@
       (effects (font (size 1.27 1.27)) hide)
     )
-    (pin "2")
-    (pin "1")
+    (pin "1")
+    (pin "2")
     (instances
       (project "GP1294-Teens4"
@@
       (effects (font (size 1.27 1.27)) hide)
     )
-    (pin "2")
-    (pin "1")
+    (pin "1")
+    (pin "2")
     (instances
       (project "GP1294-Teens4"
@@
       (effects (font (size 1.27 1.27)) hide)
     )
-    (pin "2")
-    (pin "1")
+    (pin "1")
+    (pin "2")
     (instances
       (project "GP1294-Teens4"
@@
       (effects (font (size 1.27 1.27)) hide)
     )
-    (pin "2")
-    (pin "1")
+    (pin "1")
+    (pin "2")
     (instances
       (project "GP1294-Teens4"
@@
       (effects (font (size 1.27 1.27)) hide)
     )
-    (pin "2")
-    (pin "1")
+    (pin "1")
+    (pin "2")
     (instances
       (project "GP1294-Teens4"
@@
       (effects (font (size 1.27 1.27)) hide)
     )
-    (pin "2")
-    (pin "1")
+    (pin "1")
+    (pin "2")
     (instances
       (project "GP1294-Teens4"
@@
       (effects (font (size 1.27 1.27)) hide)
     )
-    (pin "2")
-    (pin "1")
+    (pin "1")
+    (pin "2")
     (instances
       (project "GP1294-Teens4"
@@
       (effects (font (size 1.27 1.27)) hide)
     )
-    (pin "2")
-    (pin "1")
+    (pin "1")
+    (pin "2")
     (instances
       (project "GP1294-Teens4"
@@
       (effects (font (size 1.27 1.27)) hide)
     )
-    (pin "2")
-    (pin "1")
+    (pin "1")
+    (pin "2")
     (instances
       (project "GP1294-Teens4"
@@
       (effects (font (size 1.27 1.27)) hide)
     )
-    (pin "2")
-    (pin "1")
-    (instances
-      (project "GP1294-Teens4"
+    (pin "1")
+    (pin "2")
+    (instances
+      (project "GP1294-Teens4"
