File: PCB-KiCad/inputs.kicad_sch (KiCad schematic)
At the start: 39 parts, among them SW1 SW_DPDT_x2, SW2 SW_DPDT_x2, SW3 SW_DPDT_x2, SW4 SW_DPDT_x2, SW5 SW_DPDT_x2, U5 ATtiny84A-P, U6 74HC165, U7 74HC165

Commit message: Some silkscreen fixes.
Parts:
- renumbered TP24 to PA0, TP23 to PA1, TP22 to PA2, TP21 to PA3, TP20 to PB0, TP19 to PB1, TP18 to PB2, TP17 to PB3
Changed lines of the file:
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@@
   (symbol (lib_id "Connector:TestPoint") (at 190.5 91.44 90) (unit 1)
     (in_bom yes) (on_board yes) (dnp no)
-    (property "Reference" "TP22" (at 185.166 91.694 90)
+    (property "Reference" "PA2" (at 185.166 91.694 90)
       (effects (font (size 1.27 1.27)) (justify left) hide)
     )
@@
       (project "GP1294-Teens4"
         (path "/3de011e3-f89b-42a8-8637-1f4c3f0867fa/22524900-8213-405c-bbea-0973cfe551dd"
-          (reference "TP22") (unit 1)
+          (reference "PA2") (unit 1)
         )
       )
@@
   (symbol (lib_id "Connector:TestPoint") (at 190.5 88.9 90) (unit 1)
     (in_bom yes) (on_board yes) (dnp no)
-    (property "Reference" "TP23" (at 185.166 89.154 90)
+    (property "Reference" "PA1" (at 185.166 89.154 90)
       (effects (font (size 1.27 1.27)) (justify left) hide)
     )
@@
       (project "GP1294-Teens4"
         (path "/3de011e3-f89b-42a8-8637-1f4c3f0867fa/22524900-8213-405c-bbea-0973cfe551dd"
-          (reference "TP23") (unit 1)
+          (reference "PA1") (unit 1)
         )
       )
@@
   (symbol (lib_id "Connector:TestPoint") (at 190.5 93.98 90) (unit 1)
     (in_bom yes) (on_board yes) (dnp no)
-    (property "Reference" "TP21" (at 185.166 94.234 90)
+    (property "Reference" "PA3" (at 185.166 94.234 90)
       (effects (font (size 1.27 1.27)) (justify left) hide)
     )
@@
       (project "GP1294-Teens4"
         (path "/3de011e3-f89b-42a8-8637-1f4c3f0867fa/22524900-8213-405c-bbea-0973cfe551dd"
-          (reference "TP21") (unit 1)
+          (reference "PA3") (unit 1)
         )
       )
@@
   (symbol (lib_id "Connector:TestPoint") (at 190.5 116.84 90) (unit 1)
     (in_bom yes) (on_board yes) (dnp no)
-    (property "Reference" "TP17" (at 185.166 117.094 90)
+    (property "Reference" "PB3" (at 185.166 117.094 90)
       (effects (font (size 1.27 1.27)) (justify left) hide)
     )
@@
       (project "GP1294-Teens4"
         (path "/3de011e3-f89b-42a8-8637-1f4c3f0867fa/22524900-8213-405c-bbea-0973cfe551dd"
-          (reference "TP17") (unit 1)
+          (reference "PB3") (unit 1)
         )
       )
@@
   (symbol (lib_id "Connector:TestPoint") (at 190.5 111.76 90) (unit 1)
     (in_bom yes) (on_board yes) (dnp no)
-    (property "Reference" "TP19" (at 185.166 112.014 90)
+    (property "Reference" "PB1" (at 185.166 112.014 90)
       (effects (font (size 1.27 1.27)) (justify left) hide)
     )
@@
       (project "GP1294-Teens4"
         (path "/3de011e3-f89b-42a8-8637-1f4c3f0867fa/22524900-8213-405c-bbea-0973cfe551dd"
-          (reference "TP19") (unit 1)
+          (reference "PB1") (unit 1)
         )
       )
@@
   (symbol (lib_id "Connector:TestPoint") (at 190.5 86.36 90) (unit 1)
     (in_bom yes) (on_board yes) (dnp no)
-    (property "Reference" "TP24" (at 185.166 86.614 90)
+    (property "Reference" "PA0" (at 185.166 86.614 90)
       (effects (font (size 1.27 1.27)) (justify left) hide)
     )
@@
       (project "GP1294-Teens4"
         (path "/3de011e3-f89b-42a8-8637-1f4c3f0867fa/22524900-8213-405c-bbea-0973cfe551dd"
-          (reference "TP24") (unit 1)
+          (reference "PA0") (unit 1)
         )
       )
@@
   (symbol (lib_id "Connector:TestPoint") (at 190.5 109.22 90) (unit 1)
     (in_bom yes) (on_board yes) (dnp no)
-    (property "Reference" "TP20" (at 185.166 109.474 90)
+    (property "Reference" "PB0" (at 185.166 109.474 90)
       (effects (font (size 1.27 1.27)) (justify left) hide)
     )
@@
       (project "GP1294-Teens4"
         (path "/3de011e3-f89b-42a8-8637-1f4c3f0867fa/22524900-8213-405c-bbea-0973cfe551dd"
-          (reference "TP20") (unit 1)
+          (reference "PB0") (unit 1)
         )
       )
@@
   (symbol (lib_id "Connector:TestPoint") (at 190.5 114.3 90) (unit 1)
     (in_bom yes) (on_board yes) (dnp no)
-    (property "Reference" "TP18" (at 185.166 114.554 90)
+    (property "Reference" "PB2" (at 185.166 114.554 90)
       (effects (font (size 1.27 1.27)) (justify left) hide)
     )
@@
       (project "GP1294-Teens4"
         (path "/3de011e3-f89b-42a8-8637-1f4c3f0867fa/22524900-8213-405c-bbea-0973cfe551dd"
-          (reference "TP18") (unit 1)
-        )
-      )
+          (reference "PB2") (unit 1)
+        )
+      )

Commit message: Beauty fixes
Parts:
- R10: value 100 -> 4.7k
Changed lines of the file:
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@@
       (effects (font (size 1.27 1.27)) hide)
     )
-    (pin "2")
-    (pin "1")
+    (pin "1")
+    (pin "2")
     (instances
       (project "GP1294-Teens4"
@@
       (effects (font (size 1.27 1.27)) hide)
     )
-    (pin "2")
-    (pin "1")
+    (pin "1")
+    (pin "2")
     (instances
       (project "GP1294-Teens4"
@@
       (effects (font (size 1.27 1.27)))
     )
-    (property "Value" "100" (at 186.69 128.27 90)
+    (property "Value" "4.7k" (at 186.69 128.27 90)
       (effects (font (size 1.27 1.27)))
     )
@@
       (effects (font (size 1.27 1.27)) hide)
     )
-    (pin "2")
-    (pin "1")
+    (pin "1")
+    (pin "2")
     (instances
       (project "GP1294-Teens4"
@@
       (effects (font (size 1.27 1.27)) hide)
     )
-    (pin "2")
-    (pin "1")
+    (pin "1")
+    (pin "2")
     (instances
       (project "GP1294-Teens4"
@@
       (effects (font (size 1.27 1.27)) hide)
     )
-    (pin "2")
-    (pin "1")
+    (pin "1")
+    (pin "2")
     (instances
       (project "GP1294-Teens4"
@@
       (effects (font (size 1.27 1.27)) hide)
     )
-    (pin "2")
-    (pin "1")
+    (pin "1")
+    (pin "2")
     (instances
       (project "GP1294-Teens4"
@@
       (effects (font (size 1.27 1.27)) hide)
     )
-    (pin "2")
-    (pin "1")
+    (pin "1")
+    (pin "2")
     (instances
       (project "GP1294-Teens4"
@@
       (effects (font (size 1.27 1.27)) hide)
     )
-    (pin "2")
-    (pin "1")
+    (pin "1")
+    (pin "2")
     (instances
       (project "GP1294-Teens4"
@@
       (effects (font (size 1.27 1.27)) hide)
     )
-    (pin "2")
-    (pin "1")
+    (pin "1")
+    (pin "2")
     (instances
       (project "GP1294-Teens4"
@@
       (effects (font (size 1.27 1.27)) hide)
     )
-    (pin "2")
-    (pin "1")
+    (pin "1")
+    (pin "2")
     (instances
       (project "GP1294-Teens4"
@@
       (effects (font (size 1.27 1.27)) hide)
     )
-    (pin "2")
-    (pin "1")
+    (pin "1")
+    (pin "2")
     (instances
       (project "GP1294-Teens4"
@@
       (effects (font (size 1.27 1.27)) hide)
     )
-    (pin "2")
-    (pin "1")
+    (pin "1")
+    (pin "2")
     (instances
       (project "GP1294-Teens4"
@@
       (effects (font (size 1.27 1.27)) hide)
     )
-    (pin "2")
-    (pin "1")
+    (pin "1")
+    (pin "2")
     (instances
       (project "GP1294-Teens4"
@@
       (effects (font (size 1.27 1.27)) hide)
     )
-    (pin "2")
-    (pin "1")
+    (pin "1")
+    (pin "2")
     (instances
       (project "GP1294-Teens4"
@@
       (effects (font (size 1.27 1.27)) hide)
     )
-    (pin "2")
-    (pin "1")
+    (pin "1")
+    (pin "2")
     (instances
       (project "GP1294-Teens4"
@@
       (effects (font (size 1.27 1.27)) hide)
     )
-    (pin "2")
-    (pin "1")
-    (instances
-      (project "GP1294-Teens4"
+    (pin "1")
+    (pin "2")
+    (instances
+      (project "GP1294-Teens4"
